Commit message: ✨ Setting finger_width (m) instead of finger_joint

File: ur_onrobot_description/urdf/standalone_onrobot_rg2_model_macro.xacro (robot description, xacro)
@@ -125,4 +125,5 @@
       <axis xyz="-1 0 0" />
       <limit lower="-0.558505" upper="0.785398" velocity="100.0" effort="1000" />
+      <mimic joint="${prefix}finger_width" multiplier="${0.85 * ((-0.558505 - 0.785398) / 0.110)}" offset="0.785398" />
     </joint>
     <xacro:finger_joints prefix="${prefix}" fingerprefix="left" reflect="1.0"/>
@@ -139,4 +140,20 @@
     <xacro:finger_joints prefix="${prefix}" fingerprefix="right" reflect="-1.0"/>
   </xacro:macro>
+  <xacro:macro name="finger_tips" params="prefix">
+    <link name="${prefix}left_finger_tip"/>
+    <link name="${prefix}right_finger_tip"/>
+    <joint name="${prefix}left_finger_tip_joint" type="fixed">
+      <origin xyz="0 0.019 0.038" rpy="0 0 0" />
+      <parent link="${prefix}left_inner_finger" />
+      <child link="${prefix}left_finger_tip" />
+    </joint>
+    <joint name="${prefix}finger_width" type="prismatic">
+      <origin xyz="0 0 0" rpy="${pi} 0 0" />
+      <parent link="${prefix}left_finger_tip" />
+      <child link="${prefix}right_finger_tip" />
+      <axis xyz="0 -1 0" />
+      <limit lower="0" upper="0.110" velocity="100.0" effort="1000" />
+    </joint>
+  </xacro:macro>
   <xacro:macro name="onrobot_rg2" params="prefix">
     <xacro:onrobot_rg2_base_link prefix="${prefix}"/>
@@ -144,4 +161,5 @@
     <xacro:finger_links prefix="${prefix}" fingerprefix="right"/>
     <xacro:finger_joint prefix="${prefix}"/>
+    <xacro:finger_tips prefix="${prefix}"/>
     <xacro:right_outer_knuckle_joint prefix="${prefix}"/>
     <xacro:onrobot_rg2_transmission prefix="${prefix}"/>

File: ur_onrobot_description/urdf/standalone_onrobot_rg6_model_macro.xacro (robot description, xacro)
@@ -124,4 +124,5 @@
       <axis xyz="-1 0 0" />
       <limit lower="-0.628319" upper="0.628319" velocity="2.0" effort="1000" />
+      <mimic joint="${prefix}finger_width" multiplier="${0.88 * ((-0.628319 - 0.628319) / 0.160)}" offset="0.628319" />
     </joint>
     <xacro:finger_joints prefix="${prefix}" fingerprefix="left" reflect="1.0"/>
@@ -138,4 +139,20 @@
     <xacro:finger_joints prefix="${prefix}" fingerprefix="right" reflect="-1.0"/>
   </xacro:macro>
+  <xacro:macro name="finger_tips" params="prefix">
+    <link name="${prefix}left_finger_tip"/>
+    <link name="${prefix}right_finger_tip"/>
+    <joint name="${prefix}left_finger_tip_joint" type="fixed">
+      <origin xyz="0 0.025 0.058" rpy="0 0 0" />
+      <parent link="${prefix}left_inner_finger" />
+      <child link="${prefix}left_finger_tip" />
+    </joint>
+    <joint name="${prefix}finger_width" type="prismatic">
+      <origin xyz="0 0 0" rpy="${pi} 0 0" />
+      <parent link="${prefix}left_finger_tip" />
+      <child link="${prefix}right_finger_tip" />
+      <axis xyz="0 -1 0" />
+      <limit lower="0" upper="0.160" velocity="100.0" effort="1000" />
+    </joint>
+  </xacro:macro>
   <xacro:macro name="onrobot_rg6" params="prefix">
     <xacro:onrobot_rg6_base_link prefix="${prefix}"/>
@@ -143,4 +160,5 @@
     <xacro:finger_links prefix="${prefix}" fingerprefix="right"/>
     <xacro:finger_joint prefix="${prefix}"/>
+    <xacro:finger_tips prefix="${prefix}"/>
     <xacro:right_outer_knuckle_joint prefix="${prefix}"/>
     <xacro:onrobot_rg6_transmission prefix="${prefix}"/>

Commit message: ✨ Added modular MoveIt config

File: ur_onrobot_description/urdf/standalone_onrobot_rg2_model_macro.xacro (robot description, xacro)
@@ -143,4 +143,5 @@
     <link name="${prefix}left_finger_tip"/>
     <link name="${prefix}right_finger_tip"/>
+    <link name="${prefix}gripper_tcp"/>
     <joint name="${prefix}left_finger_tip_joint" type="fixed">
       <origin xyz="0 0.019 0.038" rpy="0 0 0" />
@@ -154,4 +155,9 @@
       <axis xyz="0 -1 0" />
       <limit lower="0" upper="0.110" velocity="100.0" effort="1000" />
+    </joint>
+    <joint name="${prefix}tcp_joint" type="fixed">
+      <origin xyz="0 0 0.218" rpy="0 0 0" />
+      <parent link="${prefix}onrobot_rg2_base_link" />
+      <child link="${prefix}gripper_tcp" />
     </joint>
   </xacro:macro>

File: ur_onrobot_description/urdf/standalone_onrobot_rg6_model_macro.xacro (robot description, xacro)
@@ -142,4 +142,5 @@
     <link name="${prefix}left_finger_tip"/>
     <link name="${prefix}right_finger_tip"/>
+    <link name="${prefix}gripper_tcp"/>
     <joint name="${prefix}left_finger_tip_joint" type="fixed">
       <origin xyz="0 0.025 0.058" rpy="0 0 0" />
@@ -153,4 +154,9 @@
       <axis xyz="0 -1 0" />
       <limit lower="0" upper="0.160" velocity="100.0" effort="1000" />
+    </joint>
+    <joint name="${prefix}tcp_joint" type="fixed">
+      <origin xyz="0 0 0.268" rpy="0 0 0" />
+      <parent link="${prefix}onrobot_rg6_base_link" />
+      <child link="${prefix}gripper_tcp" />
     </joint>
   </xacro:macro>

File: ur_onrobot_description/urdf/ur_onrobot.xacro (robot description, xacro)
@@ -3,4 +3,5 @@
   <!-- import macro -->
   <xacro:include filename="$(find ur_onrobot_description)/urdf/ur_onrobot_macro.xacro"/>
+  <xacro:arg name="cable_connector" default="true"/>
   <xacro:arg name="joint_limit_params" default="$(find ur_description)/config/$(arg robot_model)/joint_limits.yaml"/>
   <xacro:arg name="kinematics_params" default="$(find ur_description)/config/$(arg robot_model)/default_kinematics.yaml"/>

Commit message: ✨ Working Gazebo sim

File: ur_onrobot_description/urdf/standalone_onrobot_rg2_model_macro.xacro (robot description, xacro)
@@ -1,6 +1,6 @@
 <?xml version="1.0"?>
 <robot xmlns:xacro="http://ros.org/wiki/xacro">
-  <xacro:include filename="$(find onrobot_rg_description)/urdf/onrobot_rg2_transmission.xacro" />
-  <xacro:include filename="$(find onrobot_rg_description)/urdf/onrobot_rg2_gazebo.xacro" />
+  <xacro:include filename="$(find ur_onrobot_description)/urdf/onrobot_rg2_transmission_finger_width.xacro"/>
+  <xacro:include filename="$(find ur_onrobot_description)/urdf/onrobot_rg2_gazebo_finger_width.xacro"/>
   <xacro:macro name="outer_knuckle" params="prefix fingerprefix">
     <link name="${prefix}${fingerprefix}_outer_knuckle">
@@ -141,6 +141,18 @@
   </xacro:macro>
   <xacro:macro name="finger_tips" params="prefix">
-    <link name="${prefix}left_finger_tip"/>
-    <link name="${prefix}right_finger_tip"/>
+    <link name="${prefix}left_finger_tip">
+      <inertial>
+        <origin xyz="0 0 0" rpy="0 0 0"/>
+        <mass value="0.001"/>
+        <inertia ixx="1.0e-06" iyy="1.0e-06" izz="1.0e-06" ixy="0" ixz="0" iyz="0"/>
+      </inertial>
+    </link>
+    <link name="${prefix}right_finger_tip">
+      <inertial>
+        <origin xyz="0 0 0" rpy="0 0 0"/>
+        <mass value="0.001"/>
+        <inertia ixx="1.0e-06" iyy="1.0e-06" izz="1.0e-06" ixy="0" ixz="0" iyz="0"/>
+      </inertial>
+    </link>
     <link name="${prefix}gripper_tcp"/>
     <joint name="${prefix}left_finger_tip_joint" type="fixed">
@@ -154,5 +166,5 @@
       <child link="${prefix}right_finger_tip" />
       <axis xyz="0 -1 0" />
-      <limit lower="0" upper="0.110" velocity="100.0" effort="1000" />
+      <limit lower="0" upper="0.110" velocity="0.100" effort="20" />
     </joint>
     <joint name="${prefix}tcp_joint" type="fixed">
@@ -169,6 +181,6 @@
     <xacro:finger_tips prefix="${prefix}"/>
     <xacro:right_outer_knuckle_joint prefix="${prefix}"/>
-    <xacro:onrobot_rg2_transmission prefix="${prefix}"/>
-    <xacro:onrobot_rg2_gazebo prefix="${prefix}"/>
+    <xacro:onrobot_rg2_transmission_finger_width prefix="${prefix}"/>
+    <xacro:onrobot_rg2_gazebo_finger_width prefix="${prefix}"/>
   </xacro:macro>
 </robot>
